File: kicad/cc-110-usb.sch (KiCad schematic (older format))
At the start: 29 parts, among them J1 XLR4M, J2 USB2.0_C, U1 PCM2912A, X1 6MHz

Commit message: Added PCB
Parts:
- removed C16: 100u, cc-110-usb:C_6.3x7.7mm, symbol cc-110-usb:100u
- removed C4, C5: 100p, cc-110-usb:C_0603_0.9mm, symbol cc-110-usb:100p
- removed C6: 3u3, cc-110-usb:C_4.0x5.4mm, symbol cc-110-usb:3u3
- removed R10, R11, R7: 3k3, cc-110-usb:R_0603_0.5mm, symbol cc-110-usb:3k3
- added C6: 1u, cc-110-usb:C_0603_0.9mm, symbol cc-110-usb:1u
- added R10, R7: 22R, cc-110-usb:R_0603_0.5mm, symbol cc-110-usb:22R
Connections:
- net GND: now also J1.1 (MIC-), C6.2
- net at U1.11 (VCOM1): now also C6.1
- net at U1.18 (VOUTL): now also R7.1; no longer C13.1
- net at U1.22 (VOUTR): now also R10.1
- new net: C13.1, R10.2, R7.2
- no-connect marks 7 -> 9
Other:
- moved on the sheet: C13, C9, J1, R8

Commit message: Added schematic, BOM, and gerber
Parts:
- C1, C11, C14, C17, C18, C2, C3, C6, C7, C8, C9: MFG (none) -> Samsung Electro-Mechanics; Manufacturer Samsung Electro-Mechanics -> (none)
- C13: MFG (none) -> Nichicon; Manufacturer Nichicon -> (none)
- J1: MPN NC4MAH -> NC4MAH
- R1, R10, R14, R15, R2, R3, R4, R7, R8: MFG (none) -> Vishay; Manufacturer Vishay -> (none)
