File: kicad/cc-110-usb.kicad_pcb (KiCad board)
At the start: 2 copper layers, 20.3 x 29 mm, 25 parts, among them J1 XLR4M, J2 USB2.0_C, U1 PCM2912A, X1 6MHz

Commit message: Gerber review and readme update
Parts:
- J1: footprint cc-110-usb:J_NC4MAH -> cc-110-usb:J_NC4MAH_edge
Routing:
- net GND: vias 78 -> 76
